File: tsal-proto-sch.kicad_sch 21-42-12-729.kicad_sch (KiCad schematic)
At the start: 29 parts, among them J1 043045-0412, Q1 DMP2035U-7, Q3 UJ3N065080K3S, Q4 DMN2056U, Q5 AO3401A, U1 H11L1M, U2 NE555D

Commit message: TSAL_rdy4pcb
Parts:
- F1, F2: footprint Library:FUSE_BK_PCS -> Fuse:Fuse_1206_3216Metric
- Q1: footprint SOT23_DIO -> Package_TO_SOT_SMD:SOT-23
- R4: footprint (none) -> Resistor_SMD:R_0805_2012Metric_Pad1.20x1.40mm_HandSolder
Changed lines of the file:
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@@
 			)
 		)
-		(property "Footprint" "SOT23_DIO"
+		(property "Footprint" "Package_TO_SOT_SMD:SOT-23"
 			(at 111.76 86.36 0)
 			(effects
@@
 			)
 		)
-		(property "Footprint" "Library:FUSE_BK_PCS"
+		(property "Footprint" "Fuse:Fuse_1206_3216Metric"
 			(at 45.72 53.848 90)
 			(effects
@@
 			)
 		)
-		(property "Footprint" ""
+		(property "Footprint" "Resistor_SMD:R_0805_2012Metric_Pad1.20x1.40mm_HandSolder"
 			(at 166.37 43.688 90)
 			(effects
@@
 			)
 		)
-		(property "Footprint" "Library:FUSE_BK_PCS"
+		(property "Footprint" "Fuse:Fuse_1206_3216Metric"
 			(at 38.608 93.98 90)
 			(effects
