File: prototyping/tsal-pcb-24-25.kicad_pcb (KiCad board)
At the start: 2 copper layers, 87.6 x 36.8 mm, 30 parts, among them J1 043045-0412, Q1 DMP2035U-7, Q3 UJ3N065080K3S, Q4 DMN2056U, Q5 AO3401A, U1 H11L1M, U2 NE555D

Commit message: final 25-26 files
Parts:
- removed R4: 5k, Resistor_SMD:R_0805_2012Metric_Pad1.20x1.40mm_HandSolder
- added R5: 5k, Resistor_SMD:R_0805_2012Metric_Pad1.20x1.40mm_HandSolder, F.Cu at (173.5, 114.5)
- R1: value 10k -> 2k
- R8: value 10k -> 1k
- moved G*** 1.52 mm to (156.0, 110.0)
- moved R1 0.45 mm to (173.5, 112.0)
- moved R7 0.20 mm to (187.5, 101.8), turned to 0 degrees
- turned Q1 to 90 degrees
Connections:
- Q5 pad 1: unconnected-(Q5-G-Pad1) -> Net-(Q5-G)
- R7 pad 2: unconnected-(Q5-G-Pad1) -> Net-(U2-DIS)
- U2 pad 2: Net-(U2-THR) -> Net-(Q1-D)
- U2 pad 3: unconnected-(Q5-G-Pad1) -> Net-(Q5-G)
- U2 pad 7: unconnected-(Q5-G-Pad1) -> Net-(U2-DIS)
Routing:
- net Net-(Q5-G): track 0.00 -> 16.4 mm, vias 0 -> 2
- net Net-(U2-DIS): track 0.00 -> 10.3 mm, vias 0 -> 2
- net (no net): track 9.56 -> 0.00 mm
- net GLV+: track 47.1 -> 56.6 mm
- net GND: track 47.9 -> 44.2 mm, vias 0 -> 1
- net Net-(U2-THR): track 24.9 -> 26.3 mm, vias 2 -> 0
- net Net-(D2-K): track 21.9 -> 23.1 mm
- net Net-(Q1-D): track 29.3 -> 30.1 mm
- net Light+: track 19.7 -> 20.4 mm, vias 1 -> 0
- net /HV-: vias 0 -> 1
Other:
- board text added: "high volt"
- board text removed: "High volt"
