File: prototyping/tsal-pcb-24-25.kicad_sch (KiCad schematic)
At the start: 29 parts, among them J1 043045-0412, Q1 DMP2035U-7, Q3 UJ3N065080K3S, Q4 DMN2056U, Q5 AO3401A, U1 H11L1M, U2 NE555D

Commit message: final 25-26 files
Parts:
- removed R4: 5k, Resistor_SMD:R_0805_2012Metric_Pad1.20x1.40mm_HandSolder, symbol Device:R
- added R5: 5k, Resistor_SMD:R_0805_2012Metric_Pad1.20x1.40mm_HandSolder, symbol Device:R
- R1: value 10k -> 2k
- R8: value 10k -> 1k
Connections:
- net at Q5.1 (G), U2.3 (Q): no longer R7.2, U2.7 (DIS)
- net at Q1.3 (D), R8.2, U2.4 (R): now also U2.2 (TR), R5.1
- net at C4.1, R7.1, U2.6 (THR): now also R5.2; no longer U2.2 (TR)
- new net: R7.2, U2.7 (DIS)
Other:
- moved on the sheet: C1, C4, Q5, R7, U2
